Commit message: Moved neccessary files from franka description to aprs_description

File: urdf/franka/aprs_franka_macro.xacro (robot description, xacro)
@@ -6,24 +6,20 @@
     <xacro:include filename="$(find aprs_description)/urdf/franka/aprs_franka.ros2_control.xacro"/>
     <xacro:property name="initial_positions_file" default="$(find aprs_description)/config/franka_initial_positions.yaml"/>
-    <xacro:include filename="$(find franka_description)/robots/common/franka_arm.xacro" />
+    <xacro:include filename="$(find aprs_description)/urdf/franka/franka_arm.xacro" />
+    <xacro:include filename="$(find aprs_description)/urdf/franka/franka_hand.xacro" />
     <xacro:franka_arm
       arm_id="fr3"
       gazebo="false"
-      joint_limits="${xacro.load_yaml('$(find franka_description)/robots/fr3/joint_limits.yaml')}"
-      inertials="${xacro.load_yaml('$(find franka_description)/robots/fr3/inertials.yaml')}"
-      kinematics="${xacro.load_yaml('$(find franka_description)/robots/fr3/kinematics.yaml')}"
-      dynamics="${xacro.load_yaml('$(find franka_description)/robots/fr3/dynamics.yaml')}"
+      joint_limits="${xacro.load_yaml('$(find aprs_description)/config/fr3/joint_limits.yaml')}"
+      inertials="${xacro.load_yaml('$(find aprs_description)/config/fr3/inertials.yaml')}"
+      kinematics="${xacro.load_yaml('$(find aprs_description)/config/fr3/kinematics.yaml')}"
+      dynamics="${xacro.load_yaml('$(find aprs_description)/config/fr3/dynamics.yaml')}"
       connected_to="aprs_franka_base_link"
     />
-    <!-- Run franka macro
-    <xacro:franka_robot
+    <xacro:franka_hand
+      connected_to="fr3_link8"
       arm_id="fr3"
-      joint_limits="${xacro.load_yaml('$(find franka_description)/robots/fr3/joint_limits.yaml')}"
-      inertials="${xacro.load_yaml('$(find franka_description)/robots/fr3/inertials.yaml')}"
-      kinematics="${xacro.load_yaml('$(find franka_description)/robots/fr3/kinematics.yaml')}"
-      dynamics="${xacro.load_yaml('$(find franka_description)/robots/fr3/dynamics.yaml')}"
-      hand="true"
-      robot_ip="0.0.0.0">
-    </xacro:franka_robot> -->
+      inertials="${xacro.load_yaml('$(find aprs_description)/config/fr3/inertials.yaml')}">
+    </xacro:franka_hand>
     <!-- Run fanuc macro -->
     <xacro:aprs_franka_ros2_control

File: urdf/temp.urdf (robot description, URDF)
Before this commit: robot aprs_lab_robots, 13 links, 12 joints
Links:
- added link aprs_motoman_base_link
- added link base
- added link base_link
- added link base_link_inertia, mass 4.0; collision mesh filename=package://ur_description/meshes/ur10e/collision/base.stl; visual mesh filename=package://ur_description/meshes/ur10e/visual/base.dae
- added link fanuc_base_link, mass 0.1; collision mesh filename=file:///home/ubuntu/aprs_ws/install/aprs_description/share/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; visual mesh filename=file:///home/ubuntu/aprs_ws/install/aprs_description/share/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
- added link flange
- added link forearm_link, mass 3.87; collision mesh filename=package://ur_description/meshes/ur10e/collision/forearm.stl; visual mesh filename=package://ur_description/meshes/ur10e/visual/forearm.dae
- added link fr3_hand, mass 0.73; collision mesh filename=/home/ubuntu/aprs_ws/install/aprs_description/share/aprs_de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; visual mesh filename=/home/ubuntu/aprs_ws/install/aprs_description/share/aprs_de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
- added link fr3_hand_tcp
- added link fr3_leftfinger; collision box size=17.5e-3 15.2e-3 18.5e-3; collision box size=17.5e-3 7e-3 23.5e-3
- added link fr3_rightfinger; collision box size=17.5e-3 15.2e-3 18.5e-3; collision box size=17.5e-3 7e-3 23.5e-3
- added link ft_frame
- added link link_1, mass 1; collision mesh filename=file:///home/ubuntu/aprs_ws/install/aprs_description/share/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; visual mesh filename=file:///home/ubuntu/aprs_ws/install/aprs_description/share/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
- added link link_2, mass 1; collision mesh filename=file:///home/ubuntu/aprs_ws/install/aprs_description/share/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; visual mesh filename=file:///home/ubuntu/aprs_ws/install/aprs_description/share/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
- added link link_3, mass 1; collision mesh filename=file:///home/ubuntu/aprs_ws/install/aprs_description/share/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; visual mesh filename=file:///home/ubuntu/aprs_ws/install/aprs_description/share/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
- added link link_4, mass 1; collision mesh filename=file:///home/ubuntu/aprs_ws/install/aprs_description/share/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; visual mesh filename=file:///home/ubuntu/aprs_ws/install/aprs_description/share/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
- added link link_5, mass 1; collision mesh filename=file:///home/ubuntu/aprs_ws/install/aprs_description/share/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; visual mesh filename=file:///home/ubuntu/aprs_ws/install/aprs_description/share/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
- added link link_6, mass 1; collision mesh filename=file:///home/ubuntu/aprs_ws/install/aprs_description/share/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; visual mesh filename=file:///home/ubuntu/aprs_ws/install/aprs_description/share/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
- added link link_b, mass 1.0; collision mesh filename=file:///home/ubuntu/aprs_ws/install/aprs_description/share/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; visual mesh filename=file:///home/ubuntu/aprs_ws/install/aprs_description/share/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
- added link link_e, mass 1.0; collision mesh filename=file:///home/ubuntu/aprs_ws/install/aprs_description/share/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; visual mesh filename=file:///home/ubuntu/aprs_ws/install/aprs_description/share/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
- added link link_l, mass 1.0; collision mesh filename=file:///home/ubuntu/aprs_ws/install/aprs_description/share/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; visual mesh filename=file:///home/ubuntu/aprs_ws/install/aprs_description/share/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
- added link link_r, mass 1.0; collision mesh filename=file:///home/ubuntu/aprs_ws/install/aprs_description/share/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; visual mesh filename=file:///home/ubuntu/aprs_ws/install/aprs_description/share/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
- added link link_s, mass 1.0; collision mesh filename=file:///home/ubuntu/aprs_ws/install/aprs_description/share/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; visual mesh filename=file:///home/ubuntu/aprs_ws/install/aprs_description/share/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
- added link link_t, mass 1.0; collision mesh filename=file:///home/ubuntu/aprs_ws/install/aprs_description/share/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; visual mesh filename=file:///home/ubuntu/aprs_ws/install/aprs_description/share/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
- added link link_u, mass 1.0; collision mesh filename=file:///home/ubuntu/aprs_ws/install/aprs_description/share/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; visual mesh filename=file:///home/ubuntu/aprs_ws/install/aprs_description/share/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
- added link motoman_base_link, mass 1.0; collision mesh filename=file:///home/ubuntu/aprs_ws/install/aprs_description/share/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; visual mesh filename=file:///home/ubuntu/aprs_ws/install/aprs_description/share/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
- added link motoman_tool0
- added link shoulder_link, mass 7.778; collision mesh filename=package://ur_description/meshes/ur10e/collision/shoulder.stl; visual mesh filename=package://ur_description/meshes/ur10e/visual/shoulder.dae
- added link tool0
- added link upper_arm_link, mass 12.93; collision mesh filename=package://ur_description/meshes/ur10e/collision/upperarm.stl; visual mesh filename=package://ur_description/meshes/ur10e/visual/upperarm.dae
- added link wrist_1_link, mass 1.96; collision mesh filename=package://ur_description/meshes/ur10e/collision/wrist1.stl; visual mesh filename=package://ur_description/meshes/ur10e/visual/wrist1.dae
- added link wrist_2_link, mass 1.96; collision mesh filename=package://ur_description/meshes/ur10e/collision/wrist2.stl; visual mesh filename=package://ur_description/meshes/ur10e/visual/wrist2.dae
- added link wrist_3_link, mass 0.202; collision mesh filename=package://ur_description/meshes/ur10e/collision/wrist3.stl; visual mesh filename=package://ur_description/meshes/ur10e/visual/wrist3.dae
- link fr3_link0: geometry collision mesh filename=/home/ubuntu/aprs_ws/install/aprs_description/share/aprs_de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; visual mesh filename=/home/ubuntu/aprs_ws/install/aprs_description/share/aprs_de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
- link fr3_link1: geometry collision mesh filename=/home/ubuntu/aprs_ws/install/aprs_description/share/aprs_de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; visual mesh filename=/home/ubuntu/aprs_ws/install/aprs_description/share/aprs_de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
- link fr3_link2: geometry collision mesh filename=/home/ubuntu/aprs_ws/install/aprs_description/share/aprs_de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; visual mesh filename=/home/ubuntu/aprs_ws/install/aprs_description/share/aprs_de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
- link fr3_link3: geometry collision mesh filename=/home/ubuntu/aprs_ws/install/aprs_description/share/aprs_de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; visual mesh filename=/home/ubuntu/aprs_ws/install/aprs_description/share/aprs_de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
- link fr3_link4: geometry collision mesh filename=/home/ubuntu/aprs_ws/install/aprs_description/share/aprs_de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; visual mesh filename=/home/ubuntu/aprs_ws/install/aprs_description/share/aprs_de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
- link fr3_link5: geometry collision mesh filename=/home/ubuntu/aprs_ws/install/aprs_description/share/aprs_de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; visual mesh filename=/home/ubuntu/aprs_ws/install/aprs_description/share/aprs_de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
- link fr3_link6: geometry collision mesh filename=/home/ubuntu/aprs_ws/install/aprs_description/share/aprs_de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; visual mesh filename=/home/ubuntu/aprs_ws/install/aprs_description/share/aprs_de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
- link fr3_link7: geometry collision mesh filename=/home/ubuntu/aprs_ws/install/aprs_description/share/aprs_de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; visual mesh filename=/home/ubuntu/aprs_ws/install/aprs_description/share/aprs_de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
Joints:
- removed joint aprs_franka_base_link
- added joint aprs_franka_base_link_joint: type fixed, parent aprs_franka_base_link, child fr3_link0, origin xyz=0 0 0 rpy=0 0 0
- added joint base_joint: type fixed, parent aprs_ur_base_link, child base_link, origin xyz=0 0 0.05 rpy=0 0 0
- added joint base_joint_: type fixed, parent aprs_fanuc_base_link, child fanuc_base_link, origin xyz=0 0 0 rpy=0 0 0
- added joint base_link-base_fixed_joint: type fixed, parent base_link, child base, origin xyz=0 0 0 rpy=0 0 3.141592653589793
- added joint base_link-base_link_inertia: type fixed, parent base_link, child base_link_inertia, origin xyz=0 0 0 rpy=0 0 3.141592653589793
- added joint elbow_joint: type revolute, parent upper_arm_link, child forearm_link, origin xyz=-0.6127 0 0 rpy=0 0 0, axis 0 0 1, limit lower=-3.141592653589793 upper=3.141592653589793 effort=150.0 velocity=3.141592653589793
- added joint flange-tool0: type fixed, parent flange, child tool0, origin xyz=0 0 0 rpy=1.5707963267948966 0 1.5707963267948966
- added joint fr3_finger_joint1: type prismatic, parent fr3_hand, child fr3_leftfinger, origin xyz=0 0 0.0584 rpy=0 0 0, axis 0 1 0, limit lower=0.0 upper=0.04 effort=100 velocity=0.2
- added joint fr3_finger_joint2: type prismatic, parent fr3_hand, child fr3_rightfinger, origin xyz=0 0 0.0584 rpy=0 0 0, axis 0 -1 0, limit lower=0.0 upper=0.04 effort=100 velocity=0.2, mimic joint=fr3_finger_joint1
- added joint fr3_hand_joint: type fixed, parent fr3_link8, child fr3_hand, origin xyz=0 0 0 rpy=0 0 0
- added joint fr3_hand_tcp_joint: type fixed, parent fr3_hand, child fr3_hand_tcp, origin xyz=0 0 0.1034 rpy=0 0 0
- added joint joint_1: type revolute, parent fanuc_base_link, child link_1, origin xyz=0 0 0.330 rpy=0 0 0, axis 0 0 1, limit lower=-6.283185307179586 upper=6.283185307179586 effort=-1 velocity=7.85
- added joint joint_2: type revolute, parent link_1, child link_2, origin xyz=0.050 0 0 rpy=0 0 0, axis 0 1 0, limit lower=-6.283185307179586 upper=6.283185307179586 effort=-1 velocity=6.63
- added joint joint_3: type revolute, parent link_2, child link_3, origin xyz=0 0 0.330 rpy=0 0 0, axis 0 -1 0, limit lower=-6.283185307179586 upper=6.283185307179586 effort=-1 velocity=9.08
- added joint joint_4: type revolute, parent link_3, child link_4, origin xyz=0 0 0.035 rpy=0 0 0, axis -1 0 0, limit lower=-6.283185307179586 upper=6.283185307179586 effort=-1 velocity=9.6
- added joint joint_5: type revolute, parent link_4, child link_5, origin xyz=0.335 0 0 rpy=0 0 0, axis 0 -1 0, limit lower=-6.283185307179586 upper=6.283185307179586 effort=-1 velocity=9.51
- added joint joint_6: type revolute, parent link_5, child link_6, origin xyz=0.080 0 0 rpy=0 0 0, axis -1 0 0, limit lower=-6.283185307179586 upper=6.283185307179586 effort=-1 velocity=17.45
- added joint joint_b: type revolute, parent link_r, child link_b, origin xyz=0 0.181 0 rpy=0 0 0, axis 0 0 1, limit lower=-1.9198 upper=1.9198 effort=1000 velocity=3.4906
- added joint joint_e: type revolute, parent link_l, child link_e, origin xyz=0 0.247135547651375 0 rpy=0 0 0, axis 0 1 0, limit lower=-2.967 upper=2.967 effort=1000 velocity=2.2698
- added joint joint_l: type revolute, parent link_s, child link_l, origin xyz=0 0.298 0 rpy=0 0 0, axis 0 0 1, limit lower=-1.9198 upper=1.9198 effort=1000 velocity=2.2698
- added joint joint_r: type revolute, parent link_u, child link_r, origin xyz=0 0.23899999999989 0 rpy=0 0 0, axis 0 1 0, limit lower=-3.1415 upper=3.1415 effort=1000 velocity=3.4906
- added joint joint_s: type revolute, parent motoman_base_link, child link_s, origin xyz=0 0 0.112 rpy=1.5708 0 0, axis 0 1 0, limit lower=-3.1415 upper=3.1415 effort=1000 velocity=2.2698
- added joint joint_t: type revolute, parent link_b, child link_t, origin xyz=0 0.164069662461231 0.0015 rpy=0 0 0, axis 0 1 0, limit lower=-3.1415 upper=3.1415 effort=1000 velocity=7.0
- added joint joint_u: type revolute, parent link_e, child link_u, origin xyz=0 0.242864452348634 0 rpy=0 0 0, axis 0 0 1, limit lower=-2.967 upper=2.967 effort=1000 velocity=2.2698
- added joint link_t-motoman_tool0: type fixed, parent link_t, child motoman_tool0, origin xyz=0 0 0 rpy=0 0 -3.1415
- added joint motoman_base_joint: type fixed, parent aprs_motoman_base_link, child motoman_base_link, origin xyz=0 0 0 rpy=0 0 0
- added joint motoman_world_to_base: type fixed, parent world, child aprs_motoman_base_link, origin xyz=10 10 0 rpy=0 0 0
- added joint shoulder_lift_joint: type revolute, parent shoulder_link, child upper_arm_link, origin xyz=0 0 0 rpy=1.570796327 0 0, axis 0 0 1, limit lower=-6.283185307179586 upper=6.283185307179586 effort=330.0 velocity=2.0943951023931953
- added joint shoulder_pan_joint: type revolute, parent base_link_inertia, child shoulder_link, origin xyz=0 0 0.1807 rpy=0 0 0, axis 0 0 1, limit lower=-6.283185307179586 upper=6.283185307179586 effort=330.0 velocity=2.0943951023931953
- added joint wrist_1_joint: type revolute, parent forearm_link, child wrist_1_link, origin xyz=-0.57155 0 0.17415 rpy=0 0 0, axis 0 0 1, limit lower=-6.283185307179586 upper=6.283185307179586 effort=56.0 velocity=3.141592653589793
- added joint wrist_2_joint: type revolute, parent wrist_1_link, child wrist_2_link, origin xyz=0 -0.11985 -2.458164590756244e-11 rpy=1.570796327 0 0, axis 0 0 1, limit lower=-6.283185307179586 upper=6.283185307179586 effort=56.0 velocity=3.141592653589793
- added joint wrist_3-flange: type fixed, parent wrist_3_link, child flange, origin xyz=0 0 0 rpy=0 -1.5707963267948966 -1.5707963267948966
- added joint wrist_3_joint: type revolute, parent wrist_2_link, child wrist_3_link, origin xyz=0 0.11655 -2.390480459346185e-11 rpy=1.570796326589793 3.141592653589793 3.141592653589793, axis 0 0 1, limit lower=-6.283185307179586 upper=6.283185307179586 effort=56.0 velocity=3.141592653589793
- added joint wrist_3_link-ft_frame: type fixed, parent wrist_3_link, child ft_frame, origin xyz=0 0 0 rpy=3.141592653589793 0 0
- joint fanuc_world_to_base: origin xyz=0 0 0 rpy=0 0 0 -> xyz=0 10 0 rpy=0 0 0
