Commit message: Changes

File: urdf/franka/franka_cart_macro.xacro (robot description, xacro)
@@ -18,15 +18,18 @@
             <link name='x_rail'>
                 <collision>
-                    <origin xyz="0 ${x_rail_offset} ${rail_height}" rpy="0 0 0"/>
+                    <pose>-1.9601 -1.8161 1.1 0 0 0</pose>
                     <geometry>
-                    <box size="${x_rail_width} ${x_rail_length} ${rail_thickness}"/>
+                        <box>
+                            <size> 0.07 0.05 2 </size>
+                        </box>
                     </geometry>
                 </collision>
                 <visual>
-                    <origin xyz="0 ${x_rail_offset} ${rail_height}" rpy="0 0 0"/>
+                    <pose>-1.9601 -1.8161 1.1 0 0 0</pose>
                     <geometry>
-                        <box size="${x_rail_width} ${x_rail_length} ${rail_thickness}"/>
+                        <box>
+                            <size> 0.07 0.05 2 </size>
+                        </box>
                     </geometry>
-                    <material name="Grey"/>
                 </visual>
                 <inertial>
@@ -39,6 +42,5 @@
                 </inertial>
             </link>
-            <gazebo reference="x_rail">
-                <material>Gazebo/DarkGrey</material>
+            <!-- <gazebo reference="x_rail">
             </gazebo>
             <joint name="x_rail_world" type="fixed">
@@ -51,5 +53,7 @@
                 <origin xyz="0 0 0" rpy="0 0 0"/>
                 <geometry>
-                <box size="${y_rail_width} ${y_rail_length} ${rail_thickness}"/>
+                    <box>
+                        <size> 0.1 0.1 0.1 </size>
+                    </box>
                 </geometry>
             </collision>
@@ -57,7 +61,8 @@
                 <origin xyz="0 0 0" rpy="0 0 0"/>
                 <geometry>
-                <box size="${y_rail_width} ${y_rail_length} ${rail_thickness}"/>
+                    <box>
+                        <size> 0.1 0.1 0.1 </size>
+                    </box>
                 </geometry>
-                <material name="Grey"/>
             </visual>
             <inertial>
@@ -71,5 +76,4 @@
             </link>
             <gazebo reference="y_rail">
-                <material>Gazebo/GreyTransparent</material>
             </gazebo>
             <joint name="franka_cart_x_axis_joint" type="prismatic">
@@ -114,10 +118,10 @@
             <origin xyz="0 0 ${cart_height}" rpy="${pi} ${pi} ${pi/2}"/>
             <axis xyz="1 0 0"/>
-            <!--Add a 0.5m buffer for joint limits to avoid self-collisions-->
+            Add a 0.5m buffer for joint limits to avoid self-collisions
             <limit lower="${-y_rail_length / 2 + .5}"
                 upper="${x_rail_length / 2 - .5}"
                 velocity="1"
                 effort="100000"/>
-            </joint>
+            </joint> -->
     </xacro:macro>
 </robot>
