Commit message: Working

File: urdf/aprs_lab_robots.urdf.xacro (robot description, xacro)
@@ -4,4 +4,5 @@
   <link name="aprs_ur_base_link"/>
   <link name="aprs_fanuc_base_link"/>
+  <link name="aprs_motoman_base_link"/>
   <joint name = "ur_world_to_base" type = "fixed">
     <origin rpy = "0 0 0" xyz = "10 0 0"/>
@@ -19,7 +20,13 @@
     <child link = "aprs_franka_base_link"/>
   </joint>
+  <joint name = "motoman_world_to_base" type = "fixed">
+    <origin rpy = "0 0 0" xyz = "10 10 0"/>
+    <parent link = "world"/>
+    <child link = "aprs_motoman_base_link"/>
+  </joint>
   <xacro:include filename="$(find aprs_description)/urdf/ur/aprs_ur_macro.xacro"/>
   <xacro:include filename="$(find aprs_description)/urdf/fanuc/aprs_fanuc_macro.xacro"/>
   <xacro:include filename="$(find aprs_description)/urdf/franka/aprs_franka_macro.xacro"/>
+  <xacro:include filename="$(find aprs_description)/urdf/motoman/aprs_motoman_macro.xacro"/>
     <!-- ROS2 Control Plugin -->
   <xacro:arg name="controllers" default="$(find aprs_description)/config/robot_controllers.yaml" />
@@ -31,4 +38,7 @@
   </xacro:aprs_fanuc>
   <xacro:aprs_franka></xacro:aprs_franka>
+  <xacro:aprs_motoman
+    parent="aprs_motoman_base_link">
+  </xacro:aprs_motoman>
   <gazebo>
     <plugin filename="libgz_ros2_control-system.so" name="gz_ros2_control::GazeboSimROS2ControlPlugin">

File: urdf/fanuc/fanuc_lrmate200id_macro.xacro (robot description, xacro)
@@ -3,31 +3,31 @@
   <xacro:macro name="fanuc_lrmate200id" params="parent">
     <!-- Joint 1 -->
-    <xacro:property name="joint1upper" value="1e20"/>
-    <xacro:property name="joint1lower" value="-1e20"/>
+    <xacro:property name="joint1upper" value="${2*pi}"/>
+    <xacro:property name="joint1lower" value="${-2*pi}"/>
     <xacro:property name="joint1velocity" value="7.85"/>
     <xacro:property name="joint1effort" value="-1"/>
     <!-- Joint 2 -->
-    <xacro:property name="joint2upper" value="1e20"/>
-    <xacro:property name="joint2lower" value="-1e20"/>
+    <xacro:property name="joint2upper" value="${2*pi}"/>
+    <xacro:property name="joint2lower" value="${-2*pi}"/>
     <xacro:property name="joint2velocity" value="6.63"/>
     <xacro:property name="joint2effort" value="-1"/>
     <!-- Joint 3 -->
-    <xacro:property name="joint3upper" value="1e20"/>
-    <xacro:property name="joint3lower" value="-1e20"/>
+    <xacro:property name="joint3upper" value="${2*pi}"/>
+    <xacro:property name="joint3lower" value="${-2*pi}"/>
     <xacro:property name="joint3velocity" value="9.08"/>
     <xacro:property name="joint3effort" value="-1"/>
     <!-- Joint 4 -->
-    <xacro:property name="joint4upper" value="1e20"/>
-    <xacro:property name="joint4lower" value="-1e20"/>
+    <xacro:property name="joint4upper" value="${2*pi}"/>
+    <xacro:property name="joint4lower" value="${-2*pi}"/>
     <xacro:property name="joint4velocity" value="9.60"/>
     <xacro:property name="joint4effort" value="-1"/>
     <!-- Joint 5 -->
-    <xacro:property name="joint5upper" value="1e20"/>
-    <xacro:property name="joint5lower" value="-1e20"/>
+    <xacro:property name="joint5upper" value="${2*pi}"/>
+    <xacro:property name="joint5lower" value="${-2*pi}"/>
     <xacro:property name="joint5velocity" value="9.51"/>
     <xacro:property name="joint5effort" value="-1"/>
     <!-- Joint 6 -->
-    <xacro:property name="joint6upper" value="1e20"/>
-    <xacro:property name="joint6lower" value="-1e20"/>
+    <xacro:property name="joint6upper" value="${2*pi}"/>
+    <xacro:property name="joint6lower" value="${-2*pi}"/>
     <xacro:property name="joint6velocity" value="17.45"/>
     <xacro:property name="joint6effort" value="-1"/>

Commit message: Environment updates and everything is correctly placed

File: urdf/aprs_lab_robots.urdf.xacro (robot description, xacro)
@@ -11,15 +11,15 @@
   </joint>
   <joint name = "fanuc_world_to_base" type = "fixed">
-    <origin rpy = "0 0 0" xyz = "0 10 0"/>
+    <origin rpy = "0 0 0" xyz = "-0.5222875 -0.073025 0.84455"/>
     <parent link = "world"/>
     <child link = "aprs_fanuc_base_link"/>
   </joint>
-  <joint name = "franka_world_to_base" type = "fixed">
+  <!-- <joint name = "franka_world_to_base" type = "fixed">
     <origin rpy = "0 0 0" xyz = "0 0 0"/>
     <parent link = "world"/>
     <child link = "aprs_franka_base_link"/>
-  </joint>
+  </joint> -->
   <joint name = "motoman_world_to_base" type = "fixed">
-    <origin rpy = "0 0 0" xyz = "10 10 0"/>
+    <origin rpy = "0 0 3.14159" xyz = "0.4953 -0.08255 0.84455"/>
     <parent link = "world"/>
     <child link = "aprs_motoman_base_link"/>
@@ -31,11 +31,11 @@
     <!-- ROS2 Control Plugin -->
   <xacro:arg name="controllers" default="$(find aprs_description)/config/robot_controllers.yaml" />
-  <xacro:aprs_ur
+  <!-- <xacro:aprs_ur
     parent="aprs_ur_base_link">
-  </xacro:aprs_ur>
+  </xacro:aprs_ur> -->
   <xacro:aprs_fanuc
     parent="aprs_fanuc_base_link">
   </xacro:aprs_fanuc>
-  <xacro:aprs_franka></xacro:aprs_franka>
+  <!-- <xacro:aprs_franka></xacro:aprs_franka> -->
   <xacro:aprs_motoman
     parent="aprs_motoman_base_link">

Commit message: Can now load in robots seperately or all at once. All robots move.

File: urdf/aprs_lab_robots.urdf.xacro (robot description, xacro)
@@ -6,5 +6,5 @@
   <link name="aprs_motoman_base_link"/>
   <joint name = "ur_world_to_base" type = "fixed">
-    <origin rpy = "0 0 0" xyz = "10 0 0"/>
+    <origin rpy = "0 0 0" xyz = "0.7864625 -1.375 0.8001"/>
     <parent link = "world"/>
     <child link = "aprs_ur_base_link"/>
@@ -15,9 +15,9 @@
     <child link = "aprs_fanuc_base_link"/>
   </joint>
-  <!-- <joint name = "franka_world_to_base" type = "fixed">
-    <origin rpy = "0 0 0" xyz = "0 0 0"/>
+  <joint name = "franka_world_to_base" type = "fixed">
+    <origin rpy = "0 0 0" xyz = "-1.3145625 -1.375 0.8397875"/>
     <parent link = "world"/>
     <child link = "aprs_franka_base_link"/>
-  </joint> -->
+  </joint>
   <joint name = "motoman_world_to_base" type = "fixed">
     <origin rpy = "0 0 3.14159" xyz = "0.4953 -0.08255 0.84455"/>
@@ -31,11 +31,11 @@
     <!-- ROS2 Control Plugin -->
   <xacro:arg name="controllers" default="$(find aprs_description)/config/robot_controllers.yaml" />
-  <!-- <xacro:aprs_ur
+  <xacro:aprs_ur
     parent="aprs_ur_base_link">
-  </xacro:aprs_ur> -->
+  </xacro:aprs_ur>
   <xacro:aprs_fanuc
     parent="aprs_fanuc_base_link">
   </xacro:aprs_fanuc>
-  <!-- <xacro:aprs_franka></xacro:aprs_franka> -->
+  <xacro:aprs_franka></xacro:aprs_franka>
   <xacro:aprs_motoman
     parent="aprs_motoman_base_link">
