Commit message: Franka and UR over optical table

File: urdf/aprs_franka.urdf.xacro (robot description, xacro)
@@ -3,5 +3,5 @@
   <link name="world"/>
   <joint name = "franka_world_to_base" type = "fixed">
-    <origin rpy = "0 0 0" xyz = "-1.3145625 -1.375 0.8397875"/>
+    <origin rpy = "0 0 1.57075" xyz = "0.4364625 -0.7 0.8001"/>
     <parent link = "world"/>
     <child link = "aprs_franka_base_link"/>

File: urdf/aprs_ur.urdf.xacro (robot description, xacro)
@@ -4,5 +4,5 @@
   <link name="aprs_ur_base_link"/>
   <joint name = "ur_world_to_base" type = "fixed">
-    <origin rpy = "0 0 0" xyz = "0.7864625 -1.375 0.8001"/>
+    <origin rpy = "0 0 1.57075" xyz = "-0.6 -0.7 0.7897875"/>
     <parent link = "world"/>
     <child link = "aprs_ur_base_link"/>
